File: SparkFun_Analog_MEMS_Microphone_Breakout_VM2020.sch (EAGLE design)
At the start: 10 parts

Commit message: add prod_id to mic
Parts:
- added LOGO4: SPECIAL_INSTRUCTIONS-ORDERING, SparkFun-Aesthetics:SPECIAL_INSTRUCTIONS-ORDERING
- renumbered U$1 to U1
Other:
- note added: "v10"
- note removed: "v02"
